Commit message: do depth

File: src/basic_urdf/urdf/tutorial.urdf (robot description, URDF)
Before this commit: robot Tutorial, 4 links, 3 joints
Joints:
- joint joint1: origin xyz=0.0925 0.0575 0 rpy=0 0 0.785398163 -> xyz=0.0945 0.0585 0 rpy=0 0 0.785398163
- joint joint2: origin xyz=-0.0925 -0.0575 0.0 rpy=0 0 3.926990817 -> xyz=-0.0895 -0.0635 0.0 rpy=0 0 3.926990817
- joint joint3: origin xyz=0.1275 0.0 0.0 rpy=0 0 0 -> xyz=0.143 0.0 0.0 rpy=0 0 0
